File: KiCad/Bluetooth Multimeter/Bluetooth Multimeter rev3.kicad_pcb (KiCad board)
At the start: 2 copper layers, 55 x 90 mm, 31 parts, among them J1 V/Ohm, J2 Com, J3 mA, J4 A, J5 Parallel Prot, K1 Low Range, K2 Medium Range, K3 High Range, K4 UH Range (Ohm Only), K5 V/Ohm Switch, U1 ItsyBitsy_NRF52840_Big

Commit message: added rev 4 of PCB, should be shoppable if footprints are correct
Parts:
- moved D9 15.1 mm to (220.2, 82.0), turned to 0 degrees
- moved D4 9.91 mm to (219.3, 103.6)
- moved D3 9.91 mm to (216.0, 93.5)
Routing:
- net /V/Ohm Control: track 53.5 -> 44.4 mm
- net /A ADC In: track 80.1 -> 87.1 mm
- net GND: track 173.2 -> 168.5 mm
- net /mA ADC In: track 92.9 -> 88.6 mm
- net /Input Common: track 118.3 -> 119.4 mm
- net +3.3V: track 67.6 -> 66.7 mm
- net /Speaker Control: track 30.9 -> 31.6 mm
- net /High Range Control: track 49.4 -> 48.9 mm
