File: KiCad/Bluetooth Multimeter/Bluetooth Multimeter.kicad_pcb (KiCad board)
At the start: 2 copper layers, 55 x 90 mm, 33 parts, among them J1 V/Ohm, J2 Com, J3 mA, J4 A, J5 Parallel Prot, J6 3.3V, J7 GND, K1 Low Range, K2 Medium Range, K3 High Range, K4 UH Range (Ohm Only), K5 V/Ohm Switch, U1 ItsyBitsy_NRF52840_Big

Commit message: finalized pcb rev 4 and sent to shop
Parts:
- F1: footprint 502ProjectFootprints:LF124061_2 -> 502ProjectFootprints:LF124061_1
- F2: footprint 502ProjectFootprints:LF124041_3 -> 502ProjectFootprints:LF124041_4
- R1: footprint Resistor_THT:R_Axial_DIN0207_L6.3mm_D2.5mm_P10.16mm_Horizontal -> Resistor_THT:R_Axial_DIN0207_L6.3mm_D2.5mm_P2.54mm_Vertical
- moved RN1 22.9 mm to (122.9, 116.6), turned to 0 degrees
- moved R1 4.06 mm to (167.4, 135.4), turned to -90 degrees
- moved J1 2.54 mm to (174.2, 121.4)
- moved J4 2.54 mm to (121.4, 121.4)
- moved F1 2.50 mm to (146.8, 139.4)
- moved F2 2.23 mm to (146.0, 125.0)
- moved J2 0.25 mm to (174.0, 132.1)
Connections:
- R1 pad 1: /mA ADC In -> /Input Common
- R1 pad 2: /Input Common -> /mA ADC In
Routing:
- net Net-(K4-COM): track 17.3 -> 8.20 mm
- net /Input Common: track 118.4 -> 110.3 mm
- net /V/Ohm In: track 89.3 -> 95.6 mm
- net /mA ADC In: track 92.1 -> 96.4 mm
- net Net-(K3-COM): track 10.7 -> 6.73 mm
- net /A In: track 20.1 -> 18.6 mm
- net /A ADC In: track 80.1 -> 81.5 mm
- net Net-(K2-COM): track 6.98 -> 8.31 mm
- net /Ohm Vout: track 54.3 -> 55.3 mm
- net /mA In: track 19.2 -> 18.4 mm
